File: rx02-mega2560-pro.kicad_pcb (KiCad board)
At the start: 2 copper layers, 61.2 x 52.3 mm, 57 parts, among them J1 Conn_02x20_Odd_Even, J2 2041021-3, Q1 2N7002, Q2 2N7002, Q3 2N7002, Q4 2N7002, Q5 2N7002, Q6 2N7002, Q7 2N7002, U1 74HCT14D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

Commit message: Update to v1.2, add some more docs
Other:
- board text added: "RX02 Mega Pro v1.2 PCB by Chris Tersteeg Original by AK6DN"
- board text removed: "RX02 Mega Pro v1.1 PCB by Chris Tersteeg Original by AK6DN"
Changed lines of the file:
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@@
   )
   (paper "A4")
+  (title_block
+    (title "RX02 Mega2560 Pro")
+    (date "2023-11-12")
+    (rev "1.2")
+    (company "Chris Tersteeg")
+  )
   (layers
     (0 "F.Cu" signal)
@@
     (fp_line (start -1 -0.625) (end -1 0.625) (layer "B.Fab") (width 0.1))
     (fp_line (start -1 0.625) (end 1 0.625) (layer "B.Fab") (width 0.1))
-    (pad "1" smd roundrect (at -1 0 270) (size 1.2 1.4) (layers "B.Cu" "B.Paste" "B.Mask") (roundrect_rratio 0.208333)
+    (pad "1" smd roundrect (at -1 0 270) (size 1.2 1.4) (layers "B.Cu" "B.Paste" "B.Mask") (roundrect_rratio 0.2083333333)
       (net 105 "Net-(D4-Pad2)") (pintype "passive"))
-    (pad "2" smd roundrect (at 1 0 270) (size 1.2 1.4) (layers "B.Cu" "B.Paste" "B.Mask") (roundrect_rratio 0.208333)
+    (pad "2" smd roundrect (at 1 0 270) (size 1.2 1.4) (layers "B.Cu" "B.Paste" "B.Mask") (roundrect_rratio 0.2083333333)
       (net 1 "+5V") (pintype "passive"))
     (model "${KICAD6_3DMODEL_DIR}/Resistor_SMD.3dshapes/R_0805_2012Metric.wrl"
@@
     (fp_line (start 1 0.6) (end -0.7 0.6) (layer "B.Fab") (width 0.1))
     (fp_line (start 1 -0.6) (end 1 0.6) (layer "B.Fab") (width 0.1))
-    (pad "1" smd roundrect (at -1.025 0 270) (size 1.15 1.4) (layers "B.Cu" "B.Paste" "B.Mask") (roundrect_rratio 0.217391)
+    (pad "1" smd roundrect (at -1.025 0 270) (size 1.15 1.4) (layers "B.Cu" "B.Paste" "B.Mask") (roundrect_rratio 0.2173913043)
       (net 2 "GND") (pinfunction "K") (pintype "passive"))
-    (pad "2" smd roundrect (at 1.025 0 270) (size 1.15 1.4) (layers "B.Cu" "B.Paste" "B.Mask") (roundrect_rratio 0.217391)
+    (pad "2" smd roundrect (at 1.025 0 270) (size 1.15 1.4) (layers "B.Cu" "B.Paste" "B.Mask") (roundrect_rratio 0.2173913043)
       (net 105 "Net-(D4-Pad2)") (pinfunction "A") (pintype "passive"))
     (model "${KICAD6_3DMODEL_DIR}/LED_SMD.3dshapes/LED_0805_2012Metric.wrl"
@@
     (effects (font (size 1 1) (thickness 0.15)) (justify mirror))
   )
-  (gr_text "RX02 Mega Pro v1.1\nPCB by Chris Tersteeg\nOriginal by AK6DN" (at 154.8892 100.965) (layer "F.SilkS")
+  (gr_text "RX02 Mega Pro v1.2\nPCB by Chris Tersteeg\nOriginal by AK6DN" (at 154.8892 100.965) (layer "F.SilkS")
     (effects (font (size 0.8 0.8) (thickness 0.2)))
   )
