File: rx02-mega2560-pro.kicad_sch (KiCad schematic)
At the start: 57 parts, among them J1 Conn_02x20_Odd_Even, J2 2041021-3, Q1 2N7002, Q2 2N7002, Q3 2N7002, Q4 2N7002, Q5 2N7002, Q6 2N7002, Q7 2N7002, U1 74HCT14D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

Commit message: Update to v1.2, add some more docs
Other:
- company: (none) -> Chris Tersteeg
- title: (none) -> RX02 Mega2560 Pro
Changed lines of the file:
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@@
 (kicad_sch (version 20211123) (generator eeschema)
   (paper "A4")
+  (title_block
+    (title "RX02 Mega2560 Pro")
+    (date "2023-11-12")
+    (rev "1.2")
+    (company "Chris Tersteeg")
+  )
   (junction (at 33.02 139.7) (diameter 0) (color 0 0 0 0)
   )
